File: AMN_230V_pcb/AMN_230V_pcb.kicad_pcb (KiCad board)
At the start: 2 copper layers, 99.9 x 99.9 mm, 33 parts, among them J1 Screw_Terminal_01x03, J2 Screw_Terminal_01x03, J3 Screw_Terminal_01x03, J4 Screw_Terminal_01x04, J5 Conn_02x04_Odd_Even, K1 Relay_SPST-NO, K2 Relay_SPST-NO, K3 Relay_SPST-NO, Q1 BC817, Q2 BC817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

Commit message: 1
Parts:
- removed D5: LED, LED_SMD:LED_1206_3216Metric
- removed R8: 4k7, Resistor_SMD:R_0603_1608Metric
- added H1: MountingHole, MountingHole:MountingHole_3.5mm, F.Cu at (67.3, 83.3)
- added H2: MountingHole, MountingHole:MountingHole_3.5mm, F.Cu at (145.3, 83.3)
- added H3: MountingHole, MountingHole:MountingHole_3.5mm, F.Cu at (145.3, 119.3)
- added H4: MountingHole, MountingHole:MountingHole_3.5mm, F.Cu at (67.3, 119.3)
- added J6: Screw_Terminal_01x04, Connector_Phoenix_MC:PhoenixContact_MCV_1,5_4-G-3.5_1x04_P3.50mm_Vertical, F.Cu at (74.8, 107.0)
- added T1: TRANSF1, Library:VB-1,5_1_6, F.Cu at (110.7, 93.8)
- moved J3 168.7 mm to (132.8, 137.0), turned to 180 degrees
- moved J2 161.2 mm to (111.5, 137.0), turned to 180 degrees
- moved J1 157.0 mm to (90.2, 137.1), turned to 180 degrees
- moved V2 141.1 mm to (132.7, 127.6), turned to 180 degrees
- moved F1 136.9 mm to (114.2, 117.5), turned to 180 degrees
- moved F2 134.2 mm to (120.3, 117.7)
- moved V1 133.7 mm to (115.5, 127.7), turned to 180 degrees
- moved J5 131.2 mm to (132.8, 61.9)
- moved D2 121.8 mm to (136.6, 82.7), turned to -90 degrees
- moved D1 118.7 mm to (131.3, 82.6), turned to -90 degrees
- moved V3 115.5 mm to (101.1, 126.7), turned to 90 degrees
- moved K2 106.4 mm to (149.2, 92.5), turned to -90 degrees
- moved R5 99.1 mm to (126.9, 62.6), turned to 90 degrees
- moved R2 98.0 mm to (125.0, 62.6), turned to 90 degrees
- moved R4 96.3 mm to (121.2, 62.6), turned to 90 degrees
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Connections:
- J5 pad 1: unconnected-(J5-Pin_1-Pad1) -> GND
- J5 pad 3: Net-(J5-Pin_3) -> unconnected-(J5-Pin_3-Pad3)
- J5 pad 4: unconnected-(J5-Pin_4-Pad4) -> Net-(J5-Pin_4)
- J5 pad 5: Net-(J5-Pin_5) -> unconnected-(J5-Pin_5-Pad5)
- J5 pad 6: unconnected-(J5-Pin_6-Pad6) -> Net-(J5-Pin_6)
- J5 pad 7: Net-(J5-Pin_7) -> unconnected-(J5-Pin_7-Pad7)
- J5 pad 8: GND -> Net-(J5-Pin_8)
- R4 pad 2: Net-(J5-Pin_3) -> Net-(J5-Pin_6)
- R5 pad 2: Net-(J5-Pin_5) -> Net-(J5-Pin_4)
- R6 pad 2: Net-(J5-Pin_7) -> Net-(J5-Pin_8)
Routing:
- net +12V: track 0.00 -> 130.5 mm, vias 0 -> 2
- net Net-(J1-Pin_2): track 0.00 -> 112.8 mm
- net Net-(J1-Pin_3): track 0.00 -> 62.2 mm
- net Net-(J1-Pin_1): track 0.00 -> 53.7 mm
- net Net-(J5-Pin_8): track 0.00 -> 52.1 mm, vias 0 -> 1
- net Net-(J2-Pin_1): track 0.00 -> 42.3 mm
- net Net-(D2-A): track 0.00 -> 38.2 mm, vias 0 -> 2
- net Net-(D1-A): track 0.00 -> 38.0 mm
- net Net-(J3-Pin_1): track 0.00 -> 36.0 mm
- net Net-(F2-Pad2): track 0.00 -> 34.0 mm
- net Net-(F1-Pad2): track 0.00 -> 27.1 mm
- net Net-(J4-Pin_3): track 0.00 -> 25.0 mm
- net Net-(D4-Pad4): track 0.00 -> 23.4 mm
- net Net-(D4-Pad3): track 0.00 -> 18.3 mm
- net Net-(D4-+): track 0.00 -> 17.7 mm
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- added copper zone on B.Cu, net GND
- added copper zone on F.Cu, net GND
Other:
- board size 99.9 x 99.9 mm -> 93 x 93 mm

Commit message: 2
Parts:
- removed J5: Conn_02x04_Odd_Even, Connector_PinSocket_2.54mm:PinSocket_2x04_P2.54mm_Vertical
- added J7: Conn_02x03_Odd_Even, Connector_PinSocket_2.54mm:PinSocket_2x03_P2.54mm_Vertical, F.Cu at (132.8, 62.9)
Connections:
- J6 pad 1: unconnected-(J6-Pin_1-Pad1) -> Net-(J6-Pin_1)
- J6 pad 2: unconnected-(J6-Pin_2-Pad2) -> Net-(J6-Pin_1)
- J6 pad 3: unconnected-(J6-Pin_3-Pad3) -> +12V
- J6 pad 4: unconnected-(J6-Pin_4-Pad4) -> +12V
Routing:
- net Net-(J6-Pin_1): track 0.00 -> 96.5 mm
- net +12V: track 130.5 -> 188.9 mm
- net Net-(J7-Pin_6): track 52.1 -> 53.6 mm
- net Net-(J7-Pin_2): track 5.19 -> 3.85 mm
- net unconnected-(J5-Pin_5-Pad5): track 0.83 -> 0.00 mm
- net GND: track 0.74 -> 0.00 mm, vias 337 -> 325
- net Net-(J7-Pin_4): track 12.1 -> 11.4 mm
