File: AMN_230V_pcb/AMN_230V_pcb.kicad_sch (KiCad schematic)
At the start: 34 parts, among them J1 Screw_Terminal_01x03, J2 Screw_Terminal_01x03, J3 Screw_Terminal_01x03, J4 Screw_Terminal_01x04, J5 Conn_02x04_Odd_Even, K1 Relay_SPST-NO, K2 Relay_SPST-NO, K3 Relay_SPST-NO, Q1 BC817, Q2 BC817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

Commit message: 1
Parts:
- removed D5: LED, LED_SMD:LED_1206_3216Metric, symbol Device:LED
- removed R8: 4k7, Resistor_SMD:R_0603_1608Metric, symbol Device:R_Small
- added H1, H2, H3, H4: MountingHole, MountingHole:MountingHole_3.5mm, symbol Mechanical:MountingHole
- added J6: Screw_Terminal_01x04, Connector_Phoenix_MC:PhoenixContact_MCV_1,5_4-G-3.5_1x04_P3.50mm_Vertical, symbol Connector:Screw_Terminal_01x04
- T1: footprint LIB:VB-1,5_1_6 -> Library:VB-1,5_1_6
Connections:
- net GND: now also J5.1 (Pin_1); no longer J5.8 (Pin_8)
- net at R4.2: now also J5.6 (Pin_6); no longer J5.3 (Pin_3)
- net at R6.2: now also J5.8 (Pin_8); no longer J5.7 (Pin_7)
- net at J5.4 (Pin_4): now also R5.2
- net at J5.5 (Pin_5): no longer R5.2
Other:
- moved on the sheet: J5

Commit message: 2
Parts:
- removed J5: Conn_02x04_Odd_Even, Connector_PinSocket_2.54mm:PinSocket_2x04_P2.54mm_Vertical, symbol Connector_Generic:Conn_02x04_Odd_Even
- added J7: Conn_02x03_Odd_Even, Connector_PinSocket_2.54mm:PinSocket_2x03_P2.54mm_Vertical, symbol Connector_Generic:Conn_02x03_Odd_Even
Connections:
- net +12V: now also J6.3 (Pin_3), J6.4 (Pin_4), J7.1 (Pin_1)
- net GND: now also J7.3 (Pin_3)
- net at R4.2: now also J7.4 (Pin_4)
- net at J6.1 (Pin_1): now also J6.2 (Pin_2), J7.5 (Pin_5)
- net at R6.2: now also J7.6 (Pin_6)
- net at R5.2: now also J7.2 (Pin_2)
